Commit message: modified:   ../../bagfiles/recordGraph.py 	new file:   ../../bagfiles/trajectory_query_record 	new file:   ../../bagfiles/trajectory_record.py 	modified:   ../../kobuki_description/urdf/kobuki.urdf.xacro 	modified:   ../../kobuki_description/urdf/kobuki_gazebo.urdf.xacro

File: kobuki_description/urdf/kobuki.urdf.xacro (robot description, xacro)
@@ -10,5 +10,5 @@
   <xacro:include filename="$(find kobuki_description)/urdf/kobuki_gazebo.urdf.xacro"/>
   <!-- Kobuki -->
-  <xacro:macro name="kobuki">
+  <xacro:macro name="kobuki" params="imu_noise">
     <link name="base_footprint"/>
     <!--
@@ -238,5 +238,5 @@
         <child link="lidar_bottom"/>
      </joint>
-    <kobuki_sim/>
+    <kobuki_sim imu_n = "${imu_noise}"/>
   </xacro:macro>
 </robot>

File: kobuki_description/urdf/kobuki_gazebo.urdf.xacro (robot description, xacro)
@@ -1,5 +1,5 @@
 <?xml version="1.0"?>
 <robot name="kobuki_sim" xmlns:xacro="http://ros.org/wiki/xacro">
-  <xacro:macro name="kobuki_sim">
+  <xacro:macro name="kobuki_sim" params = "imu_n">
 	  <gazebo reference="wheel_left_link">
 	    <mu1>1.0</mu1>
@@ -203,10 +203,10 @@
       <plugin filename="libgazebo_ros_imu_sensor.so" name="imu">
         <topicName>imu</topicName>
-        <bodyName>gyro_link</bodyName>
+        <bodyName>base_footprint</bodyName>
         <updateRateHZ>10.0</updateRateHZ>
-        <gaussianNoise>${0.0014*0.0014}</gaussianNoise>
+        <gaussianNoise><!--${0.0014*0.0014}--> ${imu_n}</gaussianNoise>
         <xyzOffset>0 0 0</xyzOffset>
         <rpyOffset>0 0 0</rpyOffset>
-        <frameName>gyro_link</frameName>
+        <frameName>base_footprint</frameName>
         <initialOrientationAsReference>false</initialOrientationAsReference>
       </plugin>
