Commit message: new file:   kobuki_yd/launch/cartographer_bag_record.launch 	modified:   kobuki_yd/launch/mapping.launch 	new file:   kobuki_yd/launch/record_bag_files.launch 	new file:   kobuki_yd/launch/record_straight_line.launch 	modified:   kobuki_yd/urdf/kobuki_yd.urdf.xacro 	modified:   kobuki_yd/urdf/ydlidar.urdf.xacro

File: kobuki_yd/urdf/kobuki_yd.urdf.xacro (robot description, xacro)
@@ -1,9 +1,11 @@
 <?xml version="1.0"?>
 <robot name="kobuki_yd" xmlns:xacro="http://ros.org/wiki/xacro">
+  <xacro:arg name = "imuNoise" default = "0.00000196"/>
+  <xacro:arg name = "lidarNoise" default = "0.0014"/>
   <xacro:include filename="$(find kobuki_description)/urdf/kobuki.urdf.xacro" />
   <xacro:include filename="$(find kobuki_yd)/urdf/ydlidar.urdf.xacro" />
-  <xacro:kobuki/>
-  <ydlidar_model parent="lidar_bottom">
-    <origin xyz="0 0 0" rpy="0 0 0" />
+  <xacro:kobuki imu_noise = "$(arg imuNoise)"/>
+  <ydlidar_model parent="lidar_bottom" lidar_noise = "$(arg lidarNoise)">
+	<origin xyz="0 0 0" rpy="0 0 0" />
   </ydlidar_model>
 </robot>

File: kobuki_yd/urdf/ydlidar.urdf.xacro (robot description, xacro)
@@ -1,5 +1,5 @@
 <?xml version="1.0" ?>
-<robot xmlns:xacro="http://ros.org/wiki/xacro">
-  <xacro:macro name="ydlidar_model" params="parent *origin">
+<robot name = "ydlidar" xmlns:xacro="http://ros.org/wiki/xacro">
+  <xacro:macro name="ydlidar_model" params="parent lidar_noise *origin">
   <joint name="ydlidar_joint" type="fixed">
     <xacro:insert_block name="origin" />
@@ -116,5 +116,5 @@
                 <type>gaussian</type>
                 <mean>0.0</mean>
-                <stddev>0.004</stddev>
+                <stddev>${lidar_noise}</stddev>
               </noise>
             </ray>
